File: CANoPi.sch (EAGLE design)
At the start: 28 parts, among them IC1 ISO7242, IC2 B0505LS, U1 MCP2515(MCP2510)SS, U2 DS1307Z, U3 MCP2551, Y1 16M, Y2 32768

Commit message: Fixed the CAN GND pin issue
Parts:
- J1: device SparkFun-Connectors:CONN_023.5MM -> SparkFun-Connectors:CONN_03SCREW
Connections:
- net GND-ISO: now also J1.3
